File: pcb/dmpcb.brd (EAGLE design)
At the start: 100 x 100 mm, 1 part

Commit message: provisorische power suppy / spannungsregler
Parts:
- added AKL_PWR: (no value), con-phoenix-254:2POL254
- added C1: 0.33uF, rcl:SANYO-OSCON_A'
- added C2: 0.1uF, rcl:SANYO-OSCON_A'
- added IC1: 7805DT, linear:TO252
Connections:
- new net +5V: C2.+, IC1.2, U$1.VIN
- new net GND: AKL_PWR.2, C1.-, C2.-, IC1.3, U$1.GND@1, U$1.GND@2, U$1.GND@3
- new net V+: AKL_PWR.1, C1.+, IC1.1
Routing:
- net +5V: track 0.00 -> 57.5 mm
- net V+: track 0.00 -> 7.56 mm
- net GND: track 0.00 -> 5.10 mm, vias 0 -> 2
- added copper zone on layer 16, net GND
Changed lines of the file:
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@@
 <elements>
 <element name="U$1" library="Teensy3.1_ralfsfix" package="TEENSY3.1_ALL_RALF" value="TEENSY3.1_ALL" x="44.45" y="53.34" smashed="yes" rot="R90"/>
+<element name="AKL_PWR" library="con-phoenix-254" library_urn="urn:adsk.eagle:library:172" package="2POL254" package3d_urn="urn:adsk.eagle:package:9320/1" value="" x="13.97" y="3.81" smashed="yes">
+<attribute name="MF" value="" x="13.97" y="3.81" size="1.778" layer="27" display="off"/>
+<attribute name="MPN" value="" x="13.97" y="3.81" size="1.778" layer="27" display="off"/>
+<attribute name="NAME" x="11.176" y="5.588" size="1.27" layer="25"/>
+<attribute name="OC_FARNELL" value="unknown" x="13.97" y="3.81" size="1.778" layer="27" display="off"/>
+<attribute name="OC_NEWARK" value="unknown" x="13.97" y="3.81" size="1.778" layer="27" display="off"/>
+<attribute name="VALUE" x="11.176" y="0.762" size="1.27" layer="27"/>
+</element>
+<element name="IC1" library="linear" library_urn="urn:adsk.eagle:library:262" package="TO252" package3d_urn="urn:adsk.eagle:package:16415/2" value="7805DT" x="17.78" y="13.97" smashed="yes">
+<attribute name="NAME" x="13.97" y="11.43" size="1.27" layer="25" rot="R90"/>
+<attribute name="VALUE" x="22.86" y="11.43" size="1.27" layer="27" rot="R90"/>
+</element>
+<element name="C1" library="rcl" library_urn="urn:adsk.eagle:library:334" package="SANYO-OSCON_A'" package3d_urn="urn:adsk.eagle:package:23440/1" value="0.33uF" x="12.7" y="8.89" smashed="yes" rot="R270">
+<attribute name="NAME" x="13.97" y="10.795" size="1.27" layer="25" rot="R270"/>
+<attribute name="SPICEPREFIX" value="C" x="12.7" y="8.89" size="1.778" layer="27" rot="R270" display="off"/>
+<attribute name="VALUE" x="10.16" y="10.795" size="1.27" layer="27" rot="R270"/>
+</element>
+<element name="C2" library="rcl" library_urn="urn:adsk.eagle:library:334" package="SANYO-OSCON_A'" package3d_urn="urn:adsk.eagle:package:23440/1" value="0.1uF" x="20.32" y="5.08" smashed="yes" rot="R90">
+<attribute name="NAME" x="19.05" y="3.175" size="1.27" layer="25" rot="R90"/>
+<attribute name="SPICEPREFIX" value="C" x="20.32" y="5.08" size="1.778" layer="27" rot="R90" display="off"/>
+<attribute name="VALUE" x="22.86" y="3.175" size="1.27" layer="27" rot="R90"/>
+</element>
 </elements>
 <signals>
+<signal name="GND">
+<contactref element="U$1" pad="GND@2"/>
+<contactref element="U$1" pad="GND@3"/>
+<contactref element="U$1" pad="GND@1"/>
+<contactref element="AKL_PWR" pad="2"/>
+<contactref element="IC1" pad="3"/>
+<contactref element="C1" pad="-"/>
+<contactref element="C2" pad="-"/>
+<polygon width="0.1524" layer="16">
+<vertex x="-5.08" y="-7.62"/>
+<vertex x="113.03" y="-7.62"/>
+<vertex x="113.03" y="105.41"/>
+<vertex x="-8.89" y="105.41"/>
+<vertex x="-8.89" y="-7.62"/>
+</polygon>
+<wire x1="17.78" y1="16.47" x2="17.74" y2="16.51" width="1.27" layer="1"/>
+<wire x1="17.74" y1="16.51" x2="12.7" y2="16.51" width="1.27" layer="1"/>
+<wire x1="12.7" y1="9.64" x2="12.7" y2="16.51" width="0" layer="19" extent="1-1"/>
+<via x="12.7" y="16.51" extent="1-16" drill="0.35"/>
+<via x="12.7" y="16.51" extent="1-16" drill="0.35"/>
+</signal>
+<signal name="V+">
+<contactref element="AKL_PWR" pad="1"/>
+<contactref element="IC1" pad="1"/>
+<contactref element="C1" pad="+"/>
+<wire x1="12.7" y1="3.81" x2="12.7" y2="8.14" width="1.27" layer="16"/>
+<wire x1="15.5" y1="9.17" x2="13.73" y2="9.17" width="1.27" layer="1"/>
+<wire x1="12.7" y1="8.14" x2="13.73" y2="9.17" width="1.27" layer="1"/>
+</signal>
+<signal name="+5V">
+<contactref element="IC1" pad="2"/>
+<contactref element="U$1" pad="VIN"/>
+<contactref element="C2" pad="+"/>
+<wire x1="20.06" y1="6.09" x2="20.06" y2="9.17" width="1.27" layer="1"/>
+<wire x1="20.32" y1="5.83" x2="20.06" y2="6.09" width="1.27" layer="1"/>
+<wire x1="30.48" y1="17.05" x2="22.6" y2="9.17" width="1.27" layer="1"/>
+<wire x1="20.06" y1="9.17" x2="22.6" y2="9.17" width="1.27" layer="1"/>
+<wire x1="30.48" y1="17.05" x2="30.48" y2="52.07" width="1.27" layer="1"/>
+<wire x1="30.48" y1="52.07" x2="34.29" y2="55.88" width="1.27" layer="1"/>
+</signal>
 </signals>
 <mfgpreviewcolors>
@@
 </board>
 </drawing>
+<compatibility>
+<note version="8.2" severity="warning">
+Since Version 8.2, EAGLE supports online libraries. The ids
+of those online libraries will not be understood (or retained)
+with this version.
+</note>
+<note version="8.3" severity="warning">
+Since Version 8.3, EAGLE supports URNs for individual library
+assets (packages, symbols, and devices). The URNs of those assets
+will not be understood (or retained) with this version.
+</note>
+<note version="8.3" severity="warning">
+Since Version 8.3, EAGLE supports the association of 3D packages
+with devices in libraries, schematics, and board files. Those 3D
+packages will not be understood (or retained) with this version.
+</note>
+</compatibility>
 </eagle>
