File: pcb/dmpcb.brd (EAGLE design)
At the start: 100 x 100 mm, 63 parts, among them IC1 7805DT, IC2 L293D, IC3 MAX7219CNG, IC4 LM358D, IC5 LM358D, J7 SJ-3523-SMT-TR, Q1 IRF530, Q2 IRF530

Commit message: borading2..
Parts:
- removed AKL_PWR: (no value), con-phoenix-254:2POL254
- removed C5: 100nf, rcl:C0805
- removed C6: 10uf, rcl:PANASONIC_B
- removed IC3: MAX7219CNG, maxim:DIL24-3
- removed J3, J4: (no value), SparkFun-Connectors:1X18
- removed J5, J6: (no value), SparkFun-Connectors:1X05
- removed R14: 10k, rcl:M0805
- added 3.3V, 5V, GND: (no value), con-lstb:MA03-2
- added HOLA, HOLB, HOLC, HOLD, JP8: (no value), jumper:JP1
- added J9: (no value), SparkFun-Connectors:1X14
- added SOCKET_IN, SOCKET_OUT: (no value), con-lstb:MA05-1
- added SV1: (no value), con-lstb:MA03-1
- added SV2: (no value), con-lstb:MA08-1
- added X1: (no value), con-wago-500:W237-102
- J1: device SparkFun-Connectors:1X18 -> SparkFun-Connectors:1X11
- J2: device SparkFun-Connectors:1X18 -> SparkFun-Connectors:1X14
- moved J8 335.0 mm to (152.4, 116.8), turned to 180 degrees
- moved R18 306.4 mm to (184.2, 124.5), turned to 180 degrees
- moved R17 293.6 mm to (181.6, 115.6), turned to 180 degrees
- moved R15 285.2 mm to (181.6, 105.4), turned to 180 degrees
- moved JP6 265.5 mm to (182.9, 48.3), turned to 180 degrees
- moved IC4 264.6 mm to (264.2, 48.3), turned to 180 degrees
- moved JP5 258.5 mm to (179.1, 59.7), turned to 180 degrees
- moved JP4 252.8 mm to (152.4, -24.1), turned to 90 degrees
- moved R13 247.1 mm to (171.4, 26.7), turned to 180 degrees
- moved R12 237.1 mm to (166.4, 26.7), turned to 180 degrees
- moved R10 227.2 mm to (161.3, 26.7), turned to 180 degrees
- moved D2 222.8 mm to (157.5, 20.3), turned to 180 degrees
- moved R16 221.6 mm to (160.0, 64.8), turned to 180 degrees
- moved JP2 219.5 mm to (158.8, 34.3), turned to 180 degrees
- moved R4 217.2 mm to (156.2, 26.7), turned to 180 degrees
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Connections:
- removed net MAX7219LOAD: IC3.12, J1.8, J5.2
- removed net N$56: J4.17
- removed net N$64: J1.14
- new net MAX7219CS: SOCKET_IN.4, SV1.2, SV2.8
- net +5V: now also 5V.1, 5V.2, 5V.3, 5V.4, 5V.5, 5V.6, J2.1, SOCKET_IN.1; no longer C2.+, C5.1, C6.+, IC1.2, IC3.19, J5.5, LED1.A, R14.2
- net 3.3V: now also 3.3V.1, 3.3V.2, 3.3V.3, 3.3V.4, 3.3V.5, 3.3V.6, J2.3
- net AGND: now also J2.2
- net BETTERAUDIOOUT: now also JP8.2; no longer J4.14
- net BUTTON01: now also SV2.1; no longer J1.1
- net BUTTON02: now also SV2.2; no longer J1.2
- net DRV8825DIR: now also J1.2; no longer J1.10
- net DRV8825EN: now also J1.1; no longer J1.9
- net DRV8825RST: now also J1.4; no longer J1.12
- net DRV8825SLP: now also J1.5; no longer J1.13
- net DRV8825STEP: now also J1.3; no longer J1.11
- net GND: now also GND.1, GND.2, GND.3, GND.4, GND.5, GND.6, J9.14, SOCKET_IN.2, X1.2; no longer AKL_PWR.2, C5.2, C6.-, IC3.4, IC3.9, J5.4, J6.1, J6.2, J6.3, J6.4, J6.5
- net LM293EN: now also SV2.3; no longer J1.3
- net LM293IN01: now also SV2.4; no longer J1.4
- net LM293IN02: now also SV2.5; no longer J1.5
- net MAX7219CLK: now also SOCKET_IN.5, SV1.1, SV2.7; no longer IC3.13, J1.7, J5.1
- net MAX7219DIN: now also SOCKET_IN.3, SV1.3, SV2.6; no longer IC3.1, J1.6, J5.3
- net MOSFET01: now also J1.10; no longer J4.16
- net MOSFET02: now also J1.11; no longer J4.15
- net N$22: no longer J2.1
- net N$23: now also J2.4; no longer J2.2
- net N$25: now also C2.+, IC1.2, JP7.1, LED1.A; no longer IC3.18, R14.1
- net N$26: now also J2.5; no longer J2.3
- net N$27: now also J2.6; no longer J2.4
- net N$28: now also J2.7; no longer J2.5
- net N$29: now also J2.8; no longer J2.6
- net N$30: now also J2.9; no longer J2.7
- net N$31: now also J2.10; no longer J2.8
- net N$32: now also J2.11; no longer J2.9
- net N$33: now also J2.12; no longer J2.10
- net N$34: now also J2.13; no longer J2.11
- net N$35: now also J2.14; no longer J2.12
- net N$36: now also J9.1; no longer J2.13
- net N$37: now also J9.2; no longer J2.14
- net N$38: now also J9.3; no longer J2.15
- net N$39: now also J9.4; no longer J2.16
- net N$40: now also J9.5; no longer J2.17
- net N$41: now also J9.6; no longer J2.18
- net N$42: no longer J3.18
- net N$43: no longer J3.17
- net N$44: no longer J3.16
- net N$45: no longer J3.15
- net N$46: no longer J3.14
- net N$47: no longer J3.13
- net N$48: no longer J3.12
- net N$49: no longer J3.11
- net N$50: no longer J3.10
- net N$51: no longer J3.9
- net N$52: no longer J3.8
- net N$53: no longer J3.7
- net N$54: no longer J3.6
- net N$55: now also JP8.1; no longer J3.5
- net N$61: now also J9.12
- net N$62: now also J9.13
- net OPAMPOUT: now also J1.9; no longer J4.10
- net PIN2: now also J9.11
- net PIN3: now also J9.10; no longer J3.1
- net PIN4: now also J9.9; no longer J3.2
- net PIN5: now also J9.8; no longer J3.3
- net PIN6: now also J9.7; no longer J3.4
- net POT01: now also J1.6; no longer J4.13
- net POT02: now also J1.7; no longer J4.12
- net SENSORPORT: now also J1.8; no longer J4.11, J4.18
- net V+: now also X1.1; no longer AKL_PWR.1, JP7.1
Routing:
- net +5V: track 0.00 -> 117.5 mm, vias 0 -> 1
- net 3.3V: track 0.00 -> 49.5 mm
- net PIN6: track 0.00 -> 9.25 mm
- net PIN5: track 0.00 -> 9.25 mm
- net PIN4: track 0.00 -> 9.25 mm
- net PIN3: track 0.00 -> 9.25 mm
- net PIN2: track 0.00 -> 9.25 mm
- net N$62: track 0.00 -> 9.25 mm
- net N$61: track 0.00 -> 9.25 mm
- net N$41: track 0.00 -> 9.25 mm
- net N$40: track 0.00 -> 9.25 mm
- net N$39: track 0.00 -> 9.25 mm
- net N$38: track 0.00 -> 9.25 mm
- net N$37: track 0.00 -> 9.25 mm
- net N$36: track 0.00 -> 9.25 mm
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- added copper zone on layer 16, net GND
