File: pcb/dmpcb.sch (EAGLE design)
At the start: 1 part

Commit message: provisorische power suppy / spannungsregler
Parts:
- added AKL_PWR: (no value), con-phoenix-254:MPT2
- added C1: 0.33uF, rcl:CPOL-EUSANYO_A'
- added C2: 0.1uF, rcl:CPOL-EUSANYO_A'
- added IC1: 7805DT, linear:7805DT
Connections:
- new net +5V: C2.+, IC1.VO, U$1.VIN
- new net GND: AKL_PWR-2.1, C1.-, C2.-, IC1.GND, U$1.GND
- new net V+: AKL_PWR-1.1, C1.+, IC1.VI
Other:
- note added: "INPUT 7 - 20 Volt"
- note added: "MC 7805 CDTG (1A)"
- note added: "POWER"
- note added: "TEENSY 3.2 | LC"
- note added: "am besten dann auf die rückseite mirrorn"
- note added: "dummy stecker guten rausuchen"
