File: pcb/dmpcb2.sch (EAGLE design)
At the start: 72 parts, among them IC1 7805DT, IC2 L293D, IC4 LM358D, IC5 LM358D, J7 SJ-3523-SMT-TR, Q1 IRF530, Q2 IRF530

Commit message: added support for second display, but only is possible at the time
Parts:
- removed J3: (no value), SparkFun-Connectors:CONN_08"
- removed SOCKET_OUT: (no value), con-lstb:MA05-1
- added C11: 10uf, rcl:C-EUC0805
- added C6: 100nf, rcl:C-EUC0805
- added SV1: (no value), con-lstb:MA07-1
- added SV2: (no value), SparkFun-Connectors:CONN_12
Connections:
- new net OLEDDC: SV1.6, SV2.10
- new net OLEDRES: SV1.5, SV2.11
- net +5V: now also C11.1, C6.1, SV1.2
- net BUTTON01: now also SV2.2; no longer J3.1
- net BUTTON02: now also SV2.3; no longer J3.2
- net GND: now also C11.2, C6.2, SV1.1
- net H-BRDIGE_A_02: now also SV2.6; no longer J3.5
- net H-BRIDGE_A_01: now also SV2.5; no longer J3.4
- net H-BRIDGE_A_EN: now also SV2.4; no longer J3.3
- net MAX7219CLK: now also SV1.3, SV2.8; no longer J3.7
- net MAX7219CS: now also SV1.7, SV2.9; no longer J3.8
- net MAX7219DIN: now also SV1.4, SV2.7; no longer J3.6
Other:
- note added: "MAX7219/OLED"
- note removed: "MAX7219"
- moved on the sheet: HOLC, HOLD
